File: driver.sch (KiCad schematic (older format))
At the start: 20 parts, among them Q1 Si4542DY, Q2 Si4542DY, Q3 Si4542DY, Q4 Si4542DY, U1 TMC2590

Commit message: All but the high current stuff.
Swapped T1 for T4 past opamp, moved board thermistor, moved LED resistors, Changes to probe (diode, resistor, NC jumper), added ideal diode to schematic, added fiducials, added voltage divider to UVLO
Parts:
- U1: symbol smoothieparts:TMC2590 -> smoothiev2-prime-rescue:TMC2590-smoothieparts
Changed lines of the file:
@@
 $Descr A4 11693 8268
 encoding utf-8
-Sheet 3 10
+Sheet 3 13
 Title ""
 Date ""
@@
 $EndDescr
 $Comp
-L smoothieparts:TMC2590 U1
+L smoothiev2-prime-rescue:TMC2590-smoothieparts U1
 U 1 1 60B43DE0
 P 3400 3450
