File: ethernet.sch (KiCad schematic (older format))
At the start: 29 parts, among them J4 RJ45_Hanrun_HR911105A, U1 LAN8720A, U10 TPD4E1U06DCKR, Y1 Crystal_GND24

Commit message: All but the high current stuff.
Swapped T1 for T4 past opamp, moved board thermistor, moved LED resistors, Changes to probe (diode, resistor, NC jumper), added ideal diode to schematic, added fiducials, added voltage divider to UVLO
Parts:
- J4: symbol smoothieparts:RJ45_Hanrun_HR911105A -> smoothiev2-prime-rescue:RJ45_Hanrun_HR911105A-smoothieparts
Changed lines of the file:
@@
 $Descr A4 11693 8268
 encoding utf-8
-Sheet 2 10
+Sheet 2 13
 Title ""
 Date ""
@@
 	6950 5350 7050 5350
 $Comp
-L smoothieparts:RJ45_Hanrun_HR911105A J4
+L smoothiev2-prime-rescue:RJ45_Hanrun_HR911105A-smoothieparts J4
 U 1 1 60DC8A27
 P 7450 4150
