File: inputs.sch (KiCad schematic (older format))
At the start: 67 parts, among them J21 Conn_01x02, J22 Conn_01x02, J23 Conn_01x02, J24 Conn_01x03, J25 Conn_01x03, J26 Conn_01x03, J27 Conn_01x03, J28 Conn_01x03, J29 Conn_01x03, J31 Conn_01x04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

Commit message: All but the high current stuff.
Swapped T1 for T4 past opamp, moved board thermistor, moved LED resistors, Changes to probe (diode, resistor, NC jumper), added ideal diode to schematic, added fiducials, added voltage divider to UVLO
Parts:
- added D31: D, Diodes_SMD:D_SOD-323, symbol Device:D
- JP7: footprint Jumper:SolderJumper-2_P1.3mm_Open_RoundedPad1.0x1.5mm -> kicad-footprints-master:SolderJumper-2_P1.3mm_Bridged_RoundedPad1.0x1.5mm; symbol Jumper:SolderJumper_2_Open -> Jumper:SolderJumper_2_Bridged
- R34: value 10k -> 1k
Connections:
- net 3V3_LIMIT_IN: no longer JP7.1 (A)
- net 5V_LIMIT_IN: now also JP7.1 (A)
- net at U12.1, U12.2 (-): now also RN9.5 (R4.2); no longer RN9.8 (R1.2)
- net at U12.13 (-), U12.14: now also RN9.8 (R1.2); no longer RN9.5 (R4.2)
- net at R34.1: now also D31.1 (K); no longer JP7.2 (B)
- new net: D31.2 (A), JP7.2 (B)
