File: mosfets.sch (KiCad schematic (older format))
At the start: 55 parts, among them J11 Conn_01x02, J12 Conn_01x02, J13 Conn_01x02, J14 Conn_01x02, J17 Conn_01x02, J18 Conn_01x02, J19 Conn_01x02, J20 Conn_01x02, J44 Conn_01x02, J45 Conn_01x02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

Commit message: All but the high current stuff.
Swapped T1 for T4 past opamp, moved board thermistor, moved LED resistors, Changes to probe (diode, resistor, NC jumper), added ideal diode to schematic, added fiducials, added voltage divider to UVLO
Parts:
- R80: value 10k -> 4.7k
Changed lines of the file:
@@
 $Descr A4 11693 8268
 encoding utf-8
-Sheet 7 10
+Sheet 7 13
 Title ""
 Date ""
@@
 P 1100 5900
 F 0 "R80" V 893 5900 50  0000 C CNN
-F 1 "10k" V 984 5900 50  0000 C CNN
+F 1 "4.7k" V 984 5900 50  0000 C CNN
 F 2 "Resistor_SMD:R_0402_1005Metric" V 1030 5900 50  0001 C CNN
 F 3 "~" H 1100 5900 50  0001 C CNN
